File: how2kicad.sch (KiCad schematic (older format))
At the start: 20 parts, among them J1 USB_B_Micro, J2 Conn_01x06, SW1 SW_Push, SW2 SW_SPST, U1 AMS1117-3.3, U2 ESP-12F, U3 FT230XS

Commit message: dodaj wartosci elementow
Parts:
- C1, C2, C3, C4, C5, C6: value C -> 100nF
- R1, R2, R5: value R -> 10K
- RV1: value R_POT -> 10K
Changed lines of the file:
@@
 EESchema Schematic File Version 4
+LIBS:how2kicad-cache
 EELAYER 30 0
 EELAYER END
@@
 P 2450 1550
 F 0 "C1" H 2565 1596 50  0000 L CNN
-F 1 "C" H 2565 1505 50  0000 L CNN
+F 1 "100nF" H 2565 1505 50  0000 L CNN
 F 2 "Capacitors_SMD:C_0402" H 2488 1400 50  0001 C CNN
 F 3 "~" H 2450 1550 50  0001 C CNN
@@
 P 3550 1550
 F 0 "C4" H 3665 1596 50  0000 L CNN
-F 1 "C" H 3665 1505 50  0000 L CNN
+F 1 "100nF" H 3665 1505 50  0000 L CNN
 F 2 "Capacitors_SMD:C_0402" H 3588 1400 50  0001 C CNN
 F 3 "~" H 3550 1550 50  0001 C CNN
@@
 Wire Wire Line
 	7200 3200 7200 2950
-$Comp
-L power:GND #PWR0108
-U 1 1 5E720DDE
-P 6150 4500
-F 0 "#PWR0108" H 6150 4250 50  0001 C CNN
-F 1 "GND" H 6155 4327 50  0000 C CNN
-F 2 "" H 6150 4500 50  0001 C CNN
-F 3 "" H 6150 4500 50  0001 C CNN
-	1    6150 4500
-	1    0    0    -1
-$EndComp
 Wire Wire Line
 	7200 3400 7200 3200
@@
 P 1300 5300
 F 0 "C2" H 1415 5346 50  0000 L CNN
-F 1 "C" H 1415 5255 50  0000 L CNN
+F 1 "100nF" H 1415 5255 50  0000 L CNN
 F 2 "Capacitors_SMD:C_0402" H 1338 5150 50  0001 C CNN
 F 3 "~" H 1300 5300 50  0001 C CNN
@@
 P 900 7200
 F 0 "R2" H 970 7246 50  0000 L CNN
-F 1 "R" H 970 7155 50  0000 L CNN
+F 1 "10K" H 970 7155 50  0000 L CNN
 F 2 "Resistors_SMD:R_0402" V 830 7200 50  0001 C CNN
 F 3 "~" H 900 7200 50  0001 C CNN
@@
 P 1300 7200
 F 0 "C3" H 1415 7246 50  0000 L CNN
-F 1 "C" H 1415 7155 50  0000 L CNN
+F 1 "100nF" H 1415 7155 50  0000 L CNN
 F 2 "Capacitors_SMD:C_0402" H 1338 7050 50  0001 C CNN
 F 3 "~" H 1300 7200 50  0001 C CNN
@@
 P 4600 5650
 F 0 "R5" V 4393 5650 50  0000 C CNN
-F 1 "R" V 4484 5650 50  0000 C CNN
+F 1 "10K" V 4484 5650 50  0000 C CNN
 F 2 "Resistors_SMD:R_0402" V 4530 5650 50  0001 C CNN
 F 3 "~" H 4600 5650 50  0001 C CNN
@@
 P 4900 5950
 F 0 "C6" H 5015 5996 50  0000 L CNN
-F 1 "C" H 5015 5905 50  0000 L CNN
+F 1 "100nF" H 5015 5905 50  0000 L CNN
 F 2 "Capacitors_SMD:C_0402" H 4938 5800 50  0001 C CNN
 F 3 "~" H 4900 5950 50  0001 C CNN
@@
 P 2650 3850
 F 0 "RV1" H 2581 3896 50  0000 R CNN
-F 1 "R_POT" H 2581 3805 50  0000 R CNN
+F 1 "10K" H 2581 3805 50  0000 R CNN
 F 2 "Potentiometers:Potentiometer_Alps_RK09K_Horizontal" H 2650 3850 50  0001 C CNN
 F 3 "~" H 2650 3850 50  0001 C CNN
@@
 P 900 5300
 F 0 "R1" H 970 5346 50  0000 L CNN
-F 1 "R" H 970 5255 50  0000 L CNN
+F 1 "10K" H 970 5255 50  0000 L CNN
 F 2 "Resistors_SMD:R_0402" V 830 5300 50  0001 C CNN
 F 3 "~" H 900 5300 50  0001 C CNN
@@
 P 3900 4300
 F 0 "C5" H 4015 4346 50  0000 L CNN
-F 1 "C" H 4015 4255 50  0000 L CNN
+F 1 "100nF" H 4015 4255 50  0000 L CNN
 F 2 "Capacitors_SMD:C_0402" H 3938 4150 50  0001 C CNN
 F 3 "~" H 3900 4300 50  0001 C CNN

Commit message: dodaj wartosci elementow 2: electric boogaloo
Parts:
- R3: value R -> 23K
- R4: value R -> 10K
Changed lines of the file:
@@
 P 2450 4750
 F 0 "R4" H 2520 4796 50  0000 L CNN
-F 1 "R" H 2520 4705 50  0000 L CNN
+F 1 "10K" H 2520 4705 50  0000 L CNN
 F 2 "Resistors_SMD:R_0402" V 2380 4750 50  0001 C CNN
 F 3 "~" H 2450 4750 50  0001 C CNN
@@
 P 1850 3850
 F 0 "R3" V 1643 3850 50  0000 C CNN
-F 1 "R" V 1734 3850 50  0000 C CNN
+F 1 "23K" V 1734 3850 50  0000 C CNN
 F 2 "Resistors_SMD:R_0402" V 1780 3850 50  0001 C CNN
 F 3 "~" H 1850 3850 50  0001 C CNN
